File: KiCAD/metal-detector.sch (KiCad schematic (older format))
At the start: 33 parts, among them J1 ICSP, J2 audio out, J3 plug, Q1 2N3904, SW1 power, U1 LM7805, U2 PIC10(L)F322-I/P, X1 MXO45HS

Commit message: update readme.md
Parts:
- gave numbers to parts that had none: 1
- renumbered C10 to C11, C11 to C12, C12 to C13
Changed lines of the file:
@@
 $EndComp
 $Comp
-L C C11
+L C C12
 U 1 1 5983AC44
 P 8175 4625
-F 0 "C11" H 8050 4525 50  0000 L CNN
+F 0 "C12" H 8050 4525 50  0000 L CNN
 F 1 "100nF" H 7925 4725 50  0000 L CNN
 F 2 "" H 8213 4475 50  0001 C CNN
@@
 $EndComp
 $Comp
-L GND #PWR10
+L GND #PWR11
 U 1 1 5983AD2E
 P 8175 4775
-F 0 "#PWR10" H 8175 4525 50  0001 C CNN
+F 0 "#PWR11" H 8175 4525 50  0001 C CNN
 F 1 "GND" H 8175 4625 50  0000 C CNN
 F 2 "" H 8175 4775 50  0001 C CNN
@@
 	7475 4175 7700 4175
 $Comp
-L CP C12
+L CP C13
 U 1 1 5983B4AF
 P 8575 3925
-F 0 "C12" H 8600 4025 50  0000 L CNN
+F 0 "C13" H 8600 4025 50  0000 L CNN
 F 1 "470µF" H 8600 3825 50  0000 L CNN
 F 2 "" H 8613 3775 50  0001 C CNN
@@
 $EndComp
 $Comp
-L GND #PWR11
+L GND #PWR12
 U 1 1 5983B8A2
 P 8825 4025
-F 0 "#PWR11" H 8825 3775 50  0001 C CNN
+F 0 "#PWR12" H 8825 3775 50  0001 C CNN
 F 1 "GND" H 8825 3875 50  0000 C CNN
 F 2 "" H 8825 4025 50  0001 C CNN
@@
 $EndComp
 $Comp
-L GND #PWR8
+L GND #PWR9
 U 1 1 598487B1
 P 7250 3450
-F 0 "#PWR8" H 7250 3200 50  0001 C CNN
+F 0 "#PWR9" H 7250 3200 50  0001 C CNN
 F 1 "GND" H 7250 3300 50  0000 C CNN
 F 2 "" H 7250 3450 50  0001 C CNN
@@
 	8625 4250 8625 4475
 $Comp
-L C C10
+L C C11
 U 1 1 5985202C
 P 8050 4075
-F 0 "C10" H 8075 3975 50  0000 L CNN
+F 0 "C11" H 8075 3975 50  0000 L CNN
 F 1 "100nF" H 8075 4175 50  0000 L CNN
 F 2 "" H 8088 3925 50  0001 C CNN
@@
 $EndComp
 $Comp
-L GND #PWR9
+L GND #PWR10
 U 1 1 598521D2
 P 8050 4225
-F 0 "#PWR9" H 8050 3975 50  0001 C CNN
+F 0 "#PWR10" H 8050 3975 50  0001 C CNN
 F 1 "GND" H 8050 4075 50  0000 C CNN
 F 2 "" H 8050 4225 50  0001 C CNN
@@
 L1 15cm de diamètre\n17 tours fil émaillé 22 AWG
 $Comp
-L C C?
+L C C10
 U 1 1 59870CC9
 P 6575 2350
-F 0 "C?" H 6600 2450 50  0000 L CNN
+F 0 "C10" H 6600 2450 50  0000 L CNN
 F 1 "10pF" H 6600 2250 50  0000 L CNN
 F 2 "" H 6613 2200 50  0001 C CNN
@@
 $EndComp
 $Comp
-L GND #PWR?
+L GND #PWR8
 U 1 1 59870D5F
 P 6575 2500
-F 0 "#PWR?" H 6575 2250 50  0001 C CNN
+F 0 "#PWR8" H 6575 2250 50  0001 C CNN
 F 1 "GND" H 6575 2350 50  0000 C CNN
 F 2 "" H 6575 2500 50  0001 C CNN

Commit message: change to schematic and readme.md Added power LED
Parts:
- added D2: Power, symbol LED
- added J1: power switch, symbol CONN_01X02
- added J2: power LED, symbol CONN_01X02
- added J3: detector coil, symbol CONN_01X02
- added P1, P2, P3: plug, symbol CONN_01X02_FEMALE
- added R9: 1K, symbol R
- U2: value PIC10(L)F322-I/P -> PIC10F322-I/P
- renumbered J2 to J4, J1 to J5, J3 to P4
Connections:
- net +9v: now also J1.1 (P1), J3.2 (P2), R9.1; no longer L1.1, SW1.2
- net GND: now also J2.2 (P2)
- net at C5.2, C8.2, Q1.2 (C): now also J3.1 (P1); no longer L1.2
- net at BT1.1 (+): now also J1.2 (P2); no longer SW1.1
- net detector renamed Fosc
- new net: L1.1, P3.2
- new net: L1.2, P3.1
- new net: P1.1, SW1.1
- new net: P1.2, SW1.2
- new net: J2.1 (P1), R9.2
- new net: D2.1 (K), P2.1
- new net: D2.2 (A), P2.2
Other:
- note added: "detector coil\nL1 15cm diameter\n17 turns magnet wire 22 AWG"
- note removed: "L1 15cm de diamètre\n17 tours fil émaillé 22 AWG"
- moved on the sheet: BT1, L1, SW1
Changed lines of the file:
@@
 L L L1
 U 1 1 598387F2
-P 5250 1950
-F 0 "L1" H 5200 1950 50  0000 C CNN
-F 1 "115µH" V 5325 1950 50  0000 C CNN
-F 2 "" H 5250 1950 50  0001 C CNN
-F 3 "" H 5250 1950 50  0001 C CNN
-	1    5250 1950
+P 6775 1500
+F 0 "L1" H 6725 1500 50  0000 C CNN
+F 1 "115µH" V 6850 1500 50  0000 C CNN
+F 2 "" H 6775 1500 50  0001 C CNN
+F 3 "" H 6775 1500 50  0001 C CNN
+	1    6775 1500
 	1    0    0    -1
 $EndComp
@@
 	5250 2100 5250 2250
 Wire Wire Line
-	5250 1800 5250 1550
-Wire Wire Line
-	3625 1550 5775 1550
+	5250 1550 5250 2000
+Wire Wire Line
+	2975 1550 5775 1550
 Wire Wire Line
 	5525 1850 5525 1900
@@
 	4325 2700 4325 2450
 $Comp
-L GND #PWR3
+L GND #PWR4
 U 1 1 59838BDC
 P 4325 3075
-F 0 "#PWR3" H 4325 2825 50  0001 C CNN
+F 0 "#PWR4" H 4325 2825 50  0001 C CNN
 F 1 "GND" H 4325 2925 50  0000 C CNN
 F 2 "" H 4325 3075 50  0001 C CNN
@@
 $EndComp
 $Comp
-L GND #PWR5
+L GND #PWR6
 U 1 1 59838C0C
 P 4600 3075
-F 0 "#PWR5" H 4600 2825 50  0001 C CNN
+F 0 "#PWR6" H 4600 2825 50  0001 C CNN
 F 1 "GND" H 4600 2925 50  0000 C CNN
 F 2 "" H 4600 3075 50  0001 C CNN
@@
 $EndComp
 $Comp
-L GND #PWR6
+L GND #PWR7
 U 1 1 59838C35
 P 5250 3075
-F 0 "#PWR6" H 5250 2825 50  0001 C CNN
+F 0 "#PWR7" H 5250 2825 50  0001 C CNN
 F 1 "GND" H 5250 2925 50  0000 C CNN
 F 2 "" H 5250 3075 50  0001 C CNN
@@
 L Battery BT1
 U 1 1 59838DD1
-P 2800 1800
-F 0 "BT1" H 2900 1900 50  0000 L CNN
-F 1 "9v" H 2900 1800 50  0000 L CNN
-F 2 "" V 2800 1860 50  0001 C CNN
-F 3 "" V 2800 1860 50  0001 C CNN
-	1    2800 1800
+P 2100 1750
+F 0 "BT1" H 2200 1850 50  0000 L CNN
+F 1 "9v" H 2200 1750 50  0000 L CNN
+F 2 "" V 2100 1810 50  0001 C CNN
+F 3 "" V 2100 1810 50  0001 C CNN
+	1    2100 1750
 	1    0    0    -1
 $EndComp
@@
 L SPDT SW1
 U 1 1 59838E95
-P 3400 1600
-F 0 "SW1" H 3400 1475 60  0000 C CNN
-F 1 "power" H 3400 1775 60  0000 C CNN
-F 2 "" H 3400 1600 60  0001 C CNN
-F 3 "" H 3400 1600 60  0001 C CNN
-	1    3400 1600
+P 3325 2275
+F 0 "SW1" H 3325 2150 60  0000 C CNN
+F 1 "power" H 3325 2450 60  0000 C CNN
+F 2 "" H 3325 2275 60  0001 C CNN
+F 3 "" H 3325 2275 60  0001 C CNN
+	1    3325 2275
 	1    0    0    -1
 $EndComp
 Connection ~ 4600 1550
 Wire Wire Line
-	3175 1600 2800 1600
-$Comp
-L GND #PWR1
+	2100 1550 2875 1550
+$Comp
+L GND #PWR2
 U 1 1 59838FBD
-P 2800 2050
-F 0 "#PWR1" H 2800 1800 50  0001 C CNN
-F 1 "GND" H 2800 1900 50  0000 C CNN
-F 2 "" H 2800 2050 50  0001 C CNN
-F 3 "" H 2800 2050 50  0001 C CNN
-	1    2800 2050
-	1    0    0    -1
-$EndComp
-Wire Wire Line
-	2800 2000 2800 2050
+P 2100 2000
+F 0 "#PWR2" H 2100 1750 50  0001 C CNN
+F 1 "GND" H 2100 1850 50  0000 C CNN
+F 2 "" H 2100 2000 50  0001 C CNN
+F 3 "" H 2100 2000 50  0001 C CNN
+	1    2100 2000
+	1    0    0    -1
+$EndComp
+Wire Wire Line
+	2100 1950 2100 2000
 Text Label 4400 1550 0    60   ~ 0
 +9v
-Text Notes 3450 1550 2    39   ~ 0
+Text Notes 3450 2200 2    39   ~ 0
 on
-Text Notes 3450 1675 2    39   ~ 0
+Text Notes 3375 2350 2    39   ~ 0
 off
-NoConn ~ 3625 1650
+NoConn ~ 3550 2325
 $Comp
 L R R4
@@
 P 6875 4375
 F 0 "U2" H 6425 4825 50  0000 L CNN
-F 1 "PIC10(L)F322-I/P" H 6425 4725 50  0000 L CNN
+F 1 "PIC10F322-I/P" H 6425 4725 50  0000 L CNN
 F 2 "Housings_DIP:DIP-8_W7.62mm" H 6425 4025 50  0001 L CIN
 F 3 "" H 6875 4375 50  0001 C CNN
@@
 	4725 4175 6275 4175
 $Comp
-L GND #PWR4
+L GND #PWR5
 U 1 1 5983A2C1
 P 4425 4525
-F 0 "#PWR4" H 4425 4275 50  0001 C CNN
+F 0 "#PWR5" H 4425 4275 50  0001 C CNN
 F 1 "GND" H 4425 4375 50  0000 C CNN
 F 2 "" H 4425 4525 50  0001 C CNN
@@
 	4425 4475 4425 4525
 $Comp
-L GND #PWR7
+L GND #PWR8
 U 1 1 5983A330
 P 6275 4650
-F 0 "#PWR7" H 6275 4400 50  0001 C CNN
+F 0 "#PWR8" H 6275 4400 50  0001 C CNN
 F 1 "GND" H 6275 4500 50  0000 C CNN
 F 2 "" H 6275 4650 50  0001 C CNN
@@
 Connection ~ 6275 4575
 Text Label 6575 2200 0    39   ~ 0
-detector
+Fosc
 Text Label 7475 4375 0    39   ~ 0
-detector
+Fosc
 $Comp
 L R R5
@@
 $EndComp
 $Comp
-L GND #PWR11
+L GND #PWR12
 U 1 1 5983AD2E
 P 8175 4775
-F 0 "#PWR11" H 8175 4525 50  0001 C CNN
+F 0 "#PWR12" H 8175 4525 50  0001 C CNN
 F 1 "GND" H 8175 4625 50  0000 C CNN
 F 2 "" H 8175 4775 50  0001 C CNN
@@
 PGCLK/SYSCLK
 $Comp
-L CONN_01X05 J1
+L CONN_01X05 J5
 U 1 1 5983B173
 P 5675 5175
-F 0 "J1" H 5675 5475 50  0000 C CNN
+F 0 "J5" H 5675 5475 50  0000 C CNN
 F 1 "ICSP" V 5775 5175 50  0000 C CNN
 F 2 "" H 5675 5175 50  0001 C CNN
@@
 $EndComp
 $Comp
-L CONN_01X02 J2
+L CONN_01X02 J4
 U 1 1 5983B7E5
 P 9025 3975
-F 0 "J2" H 9025 4125 50  0000 C CNN
+F 0 "J4" H 9025 4125 50  0000 C CNN
 F 1 "audio out" V 9125 3975 50  0000 C CNN
 F 2 "" H 9025 3975 50  0001 C CNN
@@
 $EndComp
 $Comp
-L GND #PWR12
+L GND #PWR13
 U 1 1 5983B8A2
 P 8825 4025
-F 0 "#PWR12" H 8825 3775 50  0001 C CNN
+F 0 "#PWR13" H 8825 3775 50  0001 C CNN
 F 1 "GND" H 8825 3875 50  0000 C CNN
 F 2 "" H 8825 4025 50  0001 C CNN
@@
 $EndComp
 $Comp
-L CONN_01X02_FEMALE J3
+L CONN_01X02_FEMALE P4
 U 1 1 5983B974
 P 9450 4050
-F 0 "J3" H 9450 4250 50  0000 C CNN
+F 0 "P4" H 9450 4250 50  0000 C CNN
 F 1 "plug" H 9525 3850 50  0000 C CNN
 F 2 "" H 9450 4150 50  0001 C CNN
@@
 $EndComp
 $Comp
-L GND #PWR9
+L GND #PWR10
 U 1 1 598487B1
 P 7250 3450
-F 0 "#PWR9" H 7250 3200 50  0001 C CNN
+F 0 "#PWR10" H 7250 3200 50  0001 C CNN
 F 1 "GND" H 7250 3300 50  0000 C CNN
 F 2 "" H 7250 3450 50  0001 C CNN
@@
 Connection ~ 3925 1550
 $Comp
-L GND #PWR2
+L GND #PWR3
 U 1 1 59849D72
 P 3925 1875
-F 0 "#PWR2" H 3925 1625 50  0001 C CNN
+F 0 "#PWR3" H 3925 1625 50  0001 C CNN
 F 1 "GND" H 3925 1725 50  0000 C CNN
 F 2 "" H 3925 1875 50  0001 C CNN
@@
 $EndComp
 $Comp
-L GND #PWR10
+L GND #PWR11
 U 1 1 598521D2
 P 8050 4225
-F 0 "#PWR10" H 8050 3975 50  0001 C CNN
+F 0 "#PWR11" H 8050 3975 50  0001 C CNN
 F 1 "GND" H 8050 4075 50  0000 C CNN
 F 2 "" H 8050 4225 50  0001 C CNN
@@
 Wire Wire Line
 	8725 3925 8825 3925
-Text Notes 4875 1450 0    39   ~ 0
-L1 15cm de diamètre\n17 tours fil émaillé 22 AWG
+Text Notes 6450 1175 0    39   ~ 0
+detector coil\nL1 15cm diameter\n17 turns magnet wire 22 AWG
 $Comp
 L C C10
@@
 $EndComp
 $Comp
-L GND #PWR8
+L GND #PWR9
 U 1 1 59870D5F
 P 6575 2500
-F 0 "#PWR8" H 6575 2250 50  0001 C CNN
+F 0 "#PWR9" H 6575 2250 50  0001 C CNN
 F 1 "GND" H 6575 2350 50  0000 C CNN
 F 2 "" H 6575 2500 50  0001 C CNN
@@
 	1    0    0    -1
 $EndComp
+$Comp
+L R R9
+U 1 1 5993023B
+P 2525 2825
+F 0 "R9" V 2605 2825 50  0000 C CNN
+F 1 "1K" V 2525 2825 50  0000 C CNN
+F 2 "" V 2455 2825 50  0001 C CNN
+F 3 "" H 2525 2825 50  0001 C CNN
+	1    2525 2825
+	1    0    0    -1
+$EndComp
+$Comp
+L LED D2
+U 1 1 59930375
+P 3675 3325
+F 0 "D2" H 3675 3425 50  0000 C CNN
+F 1 "Power" V 3675 3150 50  0000 C CNN
+F 2 "" H 3675 3325 50  0001 C CNN
+F 3 "" H 3675 3325 50  0001 C CNN
+	1    3675 3325
+	0    -1   -1   0
+$EndComp
+Text Label 2525 2675 0    39   ~ 0
++9v
+$Comp
+L CONN_01X02_FEMALE P2
+U 1 1 59931823
+P 3150 3275
+F 0 "P2" H 3150 3475 50  0000 C CNN
+F 1 "plug" H 3225 3075 50  0000 C CNN
+F 2 "" H 3150 3375 50  0001 C CNN
+F 3 "" H 3150 3375 50  0001 C CNN
+	1    3150 3275
+	-1   0    0    1
+$EndComp
+Wire Wire Line
+	3250 3175 3675 3175
+Wire Wire Line
+	3250 3375 3250 3475
+Wire Wire Line
+	3250 3475 3675 3475
+$Comp
+L CONN_01X02 J2
+U 1 1 59931CC1
+P 2725 3250
+F 0 "J2" H 2725 3400 50  0000 C CNN
+F 1 "power LED" V 2825 3250 50  0000 C CNN
+F 2 "" H 2725 3250 50  0001 C CNN
+F 3 "" H 2725 3250 50  0001 C CNN
+	1    2725 3250
+	1    0    0    -1
+$EndComp
+$Comp
+L GND #PWR1
+U 1 1 59931FC3
+P 2525 3300
+F 0 "#PWR1" H 2525 3050 50  0001 C CNN
+F 1 "GND" H 2525 3150 50  0000 C CNN
+F 2 "" H 2525 3300 50  0001 C CNN
+F 3 "" H 2525 3300 50  0001 C CNN
+	1    2525 3300
+	1    0    0    -1
+$EndComp
+Wire Wire Line
+	2525 2975 2525 3200
+$Comp
+L CONN_01X02 J3
+U 1 1 599327AC
+P 5050 2050
+F 0 "J3" H 5050 2200 50  0000 C CNN
+F 1 "detector coil" V 5150 2050 50  0000 C CNN
+F 2 "" H 5050 2050 50  0001 C CNN
+F 3 "" H 5050 2050 50  0001 C CNN
+	1    5050 2050
+	-1   0    0    1
+$EndComp
+$Comp
+L CONN_01X02_FEMALE P3
+U 1 1 59932C13
+P 6425 1450
+F 0 "P3" H 6425 1650 50  0000 C CNN
+F 1 "plug" H 6500 1250 50  0000 C CNN
+F 2 "" H 6425 1550 50  0001 C CNN
+F 3 "" H 6425 1550 50  0001 C CNN
+	1    6425 1450
+	-1   0    0    1
+$EndComp
+Wire Wire Line
+	6525 1350 6775 1350
+Wire Wire Line
+	6525 1550 6525 1650
+Wire Wire Line
+	6525 1650 6775 1650
+$Comp
+L CONN_01X02_FEMALE P1
+U 1 1 5993378D
+P 2750 2250
+F 0 "P1" H 2750 2450 50  0000 C CNN
+F 1 "plug" H 2825 2050 50  0000 C CNN
+F 2 "" H 2750 2350 50  0001 C CNN
+F 3 "" H 2750 2350 50  0001 C CNN
+	1    2750 2250
+	-1   0    0    1
+$EndComp
+Wire Wire Line
+	2850 2350 3100 2350
+Wire Wire Line
+	3100 2350 3100 2275
+Wire Wire Line
+	3550 2225 3550 2000
+Wire Wire Line
+	3550 2000 2850 2000
+Wire Wire Line
+	2850 2000 2850 2150
+$Comp
+L CONN_01X02 J1
+U 1 1 59933CD8
+P 2925 1750
+F 0 "J1" H 2925 1900 50  0000 C CNN
+F 1 "power switch" V 3025 1750 50  0000 C CNN
+F 2 "" H 2925 1750 50  0001 C CNN
+F 3 "" H 2925 1750 50  0001 C CNN
+	1    2925 1750
+	0    1    1    0
+$EndComp
 $EndSCHEMATC
